Commit message: Add files via upload

File: my_robot_description/urdf/base/mobile_base_gazebo.xacro (robot description, xacro)
@@ -2,38 +2,34 @@
 <robot xmlns:xacro="http://www.ros.org/wiki/xacro">
   <xacro:macro name="mobile_base_gazebo_plugin">
-    <gazebo>
-      <!-- ========== Diff Drive ========== -->
-      <plugin
-        filename="libgz-sim-diff-drive-system.so"
-        name="gz::sim::systems::DiffDrive">
-        <left_joint>left_wheel_joint</left_joint>
-        <right_joint>right_wheel_joint</right_joint>
-        <wheel_separation>0.26</wheel_separation>
-        <wheel_radius>0.04</wheel_radius>
-        <max_linear_velocity>0.5</max_linear_velocity>
-        <min_linear_velocity>-0.5</min_linear_velocity>
-        <max_angular_velocity>1.0</max_angular_velocity>
-        <min_angular_velocity>-1.0</min_angular_velocity>
-        <!-- ★ 使用绝对 topic -->
-        <topic>/cmd_vel</topic>
-        <odom_topic>/odom</odom_topic>
-        <tf_topic>/tf</tf_topic>
-        <frame_id>odom</frame_id>
-        <child_frame_id>base_footprint</child_frame_id>
-        <odom_publish_frequency>30</odom_publish_frequency>
-      </plugin>
-      <!-- ========== Joint States ========== -->
-      <plugin
-        filename="libgz-sim-joint-state-publisher-system.so"
-        name="gz::sim::systems::JointStatePublisher">
-        <topic>/joint_states</topic>
-      </plugin>
-      <!-- ========== Sensors ========== -->
-      <plugin
-        filename="libgz-sim-sensors-system.so"
-        name="gz::sim::systems::Sensors">
-        <render_engine>ogre2</render_engine>
-      </plugin>
-    </gazebo>
-  </xacro:macro>
+  <gazebo>
+    <plugin
+      filename="libignition-gazebo-diff-drive-system.so"
+      name="ignition::gazebo::systems::DiffDrive">
+      <left_joint>left_wheel_joint</left_joint>
+      <right_joint>right_wheel_joint</right_joint>
+      <wheel_separation>0.26</wheel_separation>
+      <wheel_radius>0.04</wheel_radius>
+      <max_linear_velocity>0.5</max_linear_velocity>
+      <min_linear_velocity>-0.5</min_linear_velocity>
+      <max_angular_velocity>1.0</max_angular_velocity>
+      <min_angular_velocity>-1.0</min_angular_velocity>
+      <topic>/cmd_vel</topic>
+      <odom_topic>/odom</odom_topic>
+      <tf_topic>/tf</tf_topic>
+      <frame_id>odom</frame_id>
+      <child_frame_id>base_footprint</child_frame_id>
+      <odom_publish_frequency>30</odom_publish_frequency>
+    </plugin>
+    <plugin
+      filename="libignition-gazebo-joint-state-publisher-system.so"
+      name="ignition::gazebo::systems::JointStatePublisher">
+      <topic>/joint_states</topic>
+    </plugin>
+    <plugin
+      filename="libignition-gazebo-sensors-system.so"
+      name="ignition::gazebo::systems::Sensors">
+      <render_engine>ogre2</render_engine>
+    </plugin>
+  </gazebo>
+</xacro:macro>
 </robot>

File: my_robot_description/urdf/sensors/lidar.xacro (robot description, xacro)
@@ -1,7 +1,5 @@
 <?xml version="1.0"?>
 <robot xmlns:xacro="http://www.ros.org/wiki/xacro">
-  <!-- ==================== 激光雷达 ==================== -->
   <xacro:macro name="lidar_sensor" params="prefix:='lidar'">
-    <!-- 激光雷达连杆 -->
     <link name="${prefix}_link">
       <visual>
@@ -10,5 +8,5 @@
           <cylinder length="0.05" radius="0.05"/>
         </geometry>
-        <material name="black"/>  <!-- 改为黑色，与底盘一致 -->
+        <material name="black"/>
       </visual>
       <collision>
@@ -20,14 +18,13 @@
       <xacro:cylinder_inertia m="0.1" r="0.05" h="0.05"/>
     </link>
-    <!-- 关节 - 安装在底盘上 -->
     <joint name="${prefix}_joint" type="fixed">
       <parent link="base_link"/>
       <child link="${prefix}_link"/>
-      <origin xyz="0 0 0.20" rpy="0 0 0"/>  <!-- 提高到0.20，避免碰撞 -->
+      <origin xyz="0 0 0.20" rpy="0 0 0"/>
     </joint>
-    <!-- Gazebo 插件：激光雷达 -->
     <gazebo reference="${prefix}_link">
-      <sensor name="${prefix}" type="ray">
-        <topic>scan</topic>
+      <sensor name="${prefix}" type="gpu_lidar">
+        <topic>/scan</topic>
+        <frame_id>${prefix}_link</frame_id>
         <pose>0 0 0 0 0 0</pose>
         <visualize>false</visualize>
@@ -48,5 +45,5 @@
           </range>
         </ray>
-        </sensor>
+      </sensor>
     </gazebo>
   </xacro:macro>
